File: LM3886-bal-no15v-th.kicad_pcb (KiCad board)
At the start: 2 copper layers, 72.5 x 42.5 mm, 31 parts, among them J1 INPUT, J2 SPEAKER, J3 POWER, U1 LM3886

Commit message: minor fixes
Parts:
- moved C11 1.25 mm to (118.2, 68.8), turned to 0 degrees
Routing:
- net GND: vias 150 -> 151

Commit message: final touches to the PCB layout
Parts:
- added J4: Vee, footprints:Terminal_.25_PCB_TAB_TE_Connectivity_P5.08mm_, F.Cu at (81.0, 88.8)
- added J5: GND, footprints:Terminal_.25_PCB_TAB_TE_Connectivity_P5.08mm_, F.Cu at (88.0, 88.8)
- added J6: Vcc, footprints:Terminal_.25_PCB_TAB_TE_Connectivity_P5.08mm_, F.Cu at (96.0, 88.8)
- added J7: SPK+, footprints:Terminal_.25_PCB_TAB_TE_Connectivity_P5.08mm_, F.Cu at (103.2, 89.5)
- added J8: GND, footprints:Terminal_.25_PCB_TAB_TE_Connectivity_P5.08mm_, F.Cu at (112.8, 89.5)
- moved J3 2.00 mm to (88.5, 88.8)
- moved J2 1.25 mm to (108.0, 89.5)
- moved J1 1.00 mm to (127.2, 91.2)
- moved L1 1.00 mm to (109.2, 76.0)
- moved C1 0.50 mm to (131.8, 59.5)
- moved C6 0.25 mm to (103.2, 66.5)
Routing:
- net Net-(C13-Pad1): track 8.35 -> 12.7 mm
- net /ICIN-: track 17.2 -> 16.7 mm
- net /ICIN+: track 20.9 -> 20.4 mm
- net GND: vias 151 -> 144
Other:
- board text added: "GND"
- board text added: "IN+"
- board text added: "IN-"
- board text added: "SPK+"
- board text added: "V+"
- board text added: "V-"

Commit message: minor fixes
Other:
- board text added: "April 2023"
- board text added: "Rev 1.0"
