File: LM3886-bal-tht.kicad_pcb (KiCad board)
At the start: 2 copper layers, 65 x 57.5 mm, 36 parts, among them J1 INPUT, J2 SPEAKER, J3 POWER, J4 Vee, J5 GND, J6 Vcc, J7 SPK+, J8 GND, U1 LM3886

Commit message: fixed IC location
Parts:
- C11: footprint footprints:C_Disc_D3.8mm_W2.6mm_P2.50mm_centered -> Capacitor_THT:C_Rect_L7.0mm_W2.5mm_P5.00mm
- moved C11 4.65 mm to (110.8, 68.8), turned to 0 degrees
- moved C1 1.77 mm to (132.2, 57.8)
- moved U1 0.75 mm to (111.8, 61.5)
- moved R8 0.50 mm to (115.2, 73.5)
Routing:
- net Net-(C13-Pad1): track 15.0 -> 19.9 mm
- net /IN-: track 9.44 -> 13.3 mm
- net /IN+: track 10.7 -> 13.3 mm
- net Net-(C12-Pad1): track 17.1 -> 19.7 mm
- net /ICIN+: track 21.3 -> 23.4 mm
- net /ICIN-: track 18.8 -> 19.7 mm
- net GND: vias 129 -> 136
