File: LM3886-bal-tht.kicad_pcb (KiCad board)
At the start: 2 copper layers, 65 x 57.5 mm, 36 parts, among them J1 INPUT, J2 SPEAKER, J3 POWER, J4 Vee, J5 GND, J6 Vcc, J7 SPK+, J8 GND, U1 LM3886

Commit message: initial commit form the tht branch
Parts:
- C11: footprint footprints:C_Disc_D3.8mm_W2.6mm_P2.50mm_centered -> Capacitor_THT:C_Rect_L7.0mm_W2.5mm_P5.00mm
- moved C11 4.65 mm to (110.8, 68.8), turned to 0 degrees
- moved C1 1.77 mm to (132.2, 57.8)
- moved U1 0.75 mm to (111.8, 61.5)
- moved R8 0.50 mm to (115.2, 73.5)
Routing:
- net Net-(C13-Pad1): track 15.0 -> 19.9 mm
- net /IN-: track 9.44 -> 13.3 mm
- net /IN+: track 10.7 -> 13.3 mm
- net Net-(C12-Pad1): track 17.1 -> 19.7 mm
- net /ICIN+: track 21.3 -> 23.4 mm
- net /ICIN-: track 18.8 -> 19.7 mm
- net GND: vias 129 -> 136

Commit message: finished pcb layout
Parts:
- C1, C4, C5: footprint footprints:C_Disc_D3.8mm_W2.6mm_P2.50mm_centered -> Capacitor_THT:C_Rect_L7.2mm_W4.5mm_P5.00mm_FKS2_FKP2_MKS2_MKP2
- moved C1 3.76 mm to (132.0, 61.5)
- moved C4 3.75 mm to (130.0, 65.8)
- moved C11 2.02 mm to (111.0, 66.8)
- moved C5 2.00 mm to (118.8, 65.8)
- moved U1 1.25 mm to (110.5, 61.5)
- moved C8 1.00 mm to (107.0, 64.2)
- moved C9 1.00 mm to (107.0, 58.5)
- moved C10 0.79 mm to (94.8, 63.0)
- moved R1 0.75 mm to (128.5, 74.5)
- moved R2 0.75 mm to (125.2, 74.5)
- moved R3 0.75 mm to (135.0, 74.5)
- moved R4 0.75 mm to (131.8, 74.5)
- moved R5 0.75 mm to (122.0, 74.5)
- moved R6 0.75 mm to (118.8, 74.5)
- moved C7 0.56 mm to (102.0, 59.5)
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Routing:
- net /ICIN+: track 23.4 -> 26.4 mm
- net Net-(C11-Pad2): track 5.00 -> 7.10 mm
- net /SIGOUT: track 20.6 -> 18.8 mm
- net /ICIN-: track 19.7 -> 21.3 mm
- net /MUTE: track 33.6 -> 32.4 mm
- net /IN+: track 13.3 -> 12.3 mm
- net Net-(C4-Pad2): track 2.92 -> 3.67 mm
- net /IN-: track 13.3 -> 12.6 mm
- net GND: vias 136 -> 144
