File: LM3886-bal-tht.sch (KiCad schematic (older format))
At the start: 36 parts, among them J1 INPUT, J2 SPEAKER, J3 POWER, J4 Vee, J5 GND, J6 Vcc, J7 SPK+, J8 GND, U1 LM3886

Commit message: finished the new board design
Parts:
- C1: footprint Capacitor_SMD:C_0805_2012Metric -> footprints:C_Disc_D3.8mm_W2.6mm_P2.50mm_centered
- R8, R9: footprint Resistor_SMD:R_2512_6332Metric -> Resistor_THT:R_Axial_DIN0614_L14.3mm_D5.7mm_P15.24mm_Horizontal
Connections:
- net GND: now also R8.2; no longer C11.2
- net SIGOUT: now also C11.1; no longer R8.1
- new net: C11.2, R8.1
Other:
- moved on the sheet: C11, R8
Changed lines of the file:
@@
 L Device:R R8
 U 1 1 64287061
-P 5050 3200
-F 0 "R8" H 5120 3246 50  0000 L CNN
-F 1 "2R7 2W" H 5120 3155 50  0000 L CNN
-F 2 "Resistor_SMD:R_2512_6332Metric" V 4980 3200 50  0001 C CNN
-F 3 "~" H 5050 3200 50  0001 C CNN
-	1    5050 3200
+P 5050 3700
+F 0 "R8" H 5120 3746 50  0000 L CNN
+F 1 "2R7 2W" H 5120 3655 50  0000 L CNN
+F 2 "Resistor_THT:R_Axial_DIN0614_L14.3mm_D5.7mm_P15.24mm_Horizontal" V 4980 3700 50  0001 C CNN
+F 3 "~" H 5050 3700 50  0001 C CNN
+	1    5050 3700
 	1    0    0    -1
 $EndComp
@@
 L Device:C C11
 U 1 1 64288129
-P 5050 3700
-F 0 "C11" H 5165 3746 50  0000 L CNN
-F 1 "100n" H 5165 3655 50  0000 L CNN
-F 2 "footprints:C_Disc_D3.8mm_W2.6mm_P2.50mm_centered" H 5088 3550 50  0001 C CNN
-F 3 "~" H 5050 3700 50  0001 C CNN
-	1    5050 3700
+P 5050 3200
+F 0 "C11" H 5165 3246 50  0000 L CNN
+F 1 "100n" H 5165 3155 50  0000 L CNN
+F 2 "footprints:C_Disc_D3.8mm_W2.6mm_P2.50mm_centered" H 5088 3050 50  0001 C CNN
+F 3 "~" H 5050 3200 50  0001 C CNN
+	1    5050 3200
 	1    0    0    -1
 $EndComp
@@
 F 0 "R9" V 5143 2900 50  0000 C CNN
 F 1 "10R 2W" V 5234 2900 50  0000 C CNN
-F 2 "Resistor_SMD:R_2512_6332Metric" V 5280 2900 50  0001 C CNN
+F 2 "Resistor_THT:R_Axial_DIN0614_L14.3mm_D5.7mm_P15.24mm_Horizontal" V 5280 2900 50  0001 C CNN
 F 3 "~" H 5350 2900 50  0001 C CNN
 	1    5350 2900
@@
 F 0 "C1" H 2685 2854 50  0000 R CNN
 F 1 "220p" H 2685 2945 50  0000 R CNN
-F 2 "Capacitor_SMD:C_0805_2012Metric" H 2838 2750 50  0001 C CNN
+F 2 "footprints:C_Disc_D3.8mm_W2.6mm_P2.50mm_centered" H 2838 2750 50  0001 C CNN
 F 3 "~" H 2800 2900 50  0001 C CNN
 	1    2800 2900

Commit message: initial commit form the tht branch
Parts:
- C11: footprint footprints:C_Disc_D3.8mm_W2.6mm_P2.50mm_centered -> Capacitor_THT:C_Rect_L7.0mm_W2.5mm_P5.00mm
Changed lines of the file:
@@
 F 0 "C11" H 5165 3246 50  0000 L CNN
 F 1 "100n" H 5165 3155 50  0000 L CNN
-F 2 "footprints:C_Disc_D3.8mm_W2.6mm_P2.50mm_centered" H 5088 3050 50  0001 C CNN
+F 2 "Capacitor_THT:C_Rect_L7.0mm_W2.5mm_P5.00mm" H 5088 3050 50  0001 C CNN
 F 3 "~" H 5050 3200 50  0001 C CNN
 	1    5050 3200

Commit message: finished pcb layout
Parts:
- C1, C4, C5: footprint footprints:C_Disc_D3.8mm_W2.6mm_P2.50mm_centered -> Capacitor_THT:C_Rect_L7.2mm_W4.5mm_P5.00mm_FKS2_FKP2_MKS2_MKP2
Changed lines of the file:
@@
 F 0 "C4" V 4050 1650 50  0000 R CNN
 F 1 "33p" V 3950 1650 50  0000 R CNN
-F 2 "footprints:C_Disc_D3.8mm_W2.6mm_P2.50mm_centered" H 3838 1450 50  0001 C CNN
+F 2 "Capacitor_THT:C_Rect_L7.2mm_W4.5mm_P5.00mm_FKS2_FKP2_MKS2_MKP2" H 3838 1450 50  0001 C CNN
 F 3 "~" H 3800 1600 50  0001 C CNN
 	1    3800 1600
@@
 F 0 "C5" V 3550 4350 50  0000 R CNN
 F 1 "33p" V 3650 4400 50  0000 R CNN
-F 2 "footprints:C_Disc_D3.8mm_W2.6mm_P2.50mm_centered" H 3838 4150 50  0001 C CNN
+F 2 "Capacitor_THT:C_Rect_L7.2mm_W4.5mm_P5.00mm_FKS2_FKP2_MKS2_MKP2" H 3838 4150 50  0001 C CNN
 F 3 "~" H 3800 4300 50  0001 C CNN
 	1    3800 4300
@@
 F 0 "C1" H 2685 2854 50  0000 R CNN
 F 1 "220p" H 2685 2945 50  0000 R CNN
-F 2 "footprints:C_Disc_D3.8mm_W2.6mm_P2.50mm_centered" H 2838 2750 50  0001 C CNN
+F 2 "Capacitor_THT:C_Rect_L7.2mm_W4.5mm_P5.00mm_FKS2_FKP2_MKS2_MKP2" H 2838 2750 50  0001 C CNN
 F 3 "~" H 2800 2900 50  0001 C CNN
 	1    2800 2900
